File: pcb/alex_solution/CircuitCapteurCardiaque.kicad_pcb (KiCad board)
At the start: 2 copper layers, 96.5 x 34.3 mm, 30 parts, among them J1 Conn_01x02, J10 Conn_Coaxial, J11 Conn_01x03, J12 Conn_01x02, J2 Conn_01x02, J4 Conn_01x01_Socket, J5 Conn_01x03_Pin, U1 LM358, U2 MAX1857EUA47+, U3 MAX1857EUA47+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

Commit message: Add last kicad + code folder
Parts:
- moved J10 11.3 mm to (118.7, 106.0)
- moved U5 5.49 mm to (153.0, 101.6)
- moved J2 2.53 mm to (111.1, 90.2)
Routing:
- net GND: track 302.6 -> 195.7 mm
- net Net-(J10-In): track 7.62 -> 20.3 mm
- net Net-(U1B--): track 26.1 -> 30.7 mm
- net Vsup: track 38.9 -> 42.3 mm
- net Net-(J2-Pin_1): track 15.7 -> 18.2 mm
- net Net-(U1A--): track 19.3 -> 21.7 mm
- net Net-(J1-Pin_1): track 19.0 -> 21.3 mm
- net VDD: track 25.1 -> 26.9 mm
- net Sensor: track 6.24 -> 4.45 mm
- net Net-(C2-Pad1): track 15.6 -> 16.7 mm
- net ADC: track 49.5 -> 48.5 mm
- net Net-(U1A-+): track 13.1 -> 13.6 mm
Other:
- board size 96.5 x 34.3 mm -> 92.7 x 54.6 mm
- board text added: "*"
- board text added: "J12"
