File: pcb/alex_solution/CircuitCapteurCardiaque.kicad_sch (KiCad schematic)
At the start: 31 parts, among them J1 Conn_01x02, J10 Conn_Coaxial, J11 Conn_01x03, J12 Conn_01x02, J2 Conn_01x02, J3 Conn_01x01_Socket, J4 Conn_01x01_Socket, J5 Conn_01x03_Pin, U1 LM358, U2 MAX1857EUA47+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

Commit message: Add last kicad + code folder
Changed lines of the file:
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@@
 	(wire
 		(pts
-			(xy 26.67 46.99) (xy 33.02 46.99)
+			(xy 25.4 46.99) (xy 33.02 46.99)
 		)
 		(stroke
@@
 	(global_label "Sensor"
 		(shape input)
-		(at 26.67 46.99 180)
+		(at 25.4 46.99 180)
 		(fields_autoplaced yes)
 		(effects
@@
 		)
 		(property "Intersheetrefs" "${INTERSHEET_REFS}"
-			(at 17.2744 46.99 0)
+			(at 16.0044 46.99 0)
 			(effects
 				(font
